Commit message: Add files via upload

File: drone_description/urdf/drone.xacro (robot description, xacro)
@@ -16,4 +16,30 @@
     <child link="base_link" />
   </joint>
+<joint name="hokuyo_joint" type="fixed">
+    <axis xyz="0 1 0" />
+    <origin xyz="0 0 0.2" rpy="0 0 0"/>
+    <parent link="base_link"/>
+    <child link="hokuyo_link"/>
+  </joint>
+  <!-- Hokuyo Laser -->
+  <link name="hokuyo_link">
+    <collision>
+      <origin xyz="0 0 0" rpy="0 0 0"/>
+      <geometry>
+    <box size="0.1 0.1 0.1"/>
+      </geometry>
+    </collision>
+    <visual>
+      <origin xyz="0 0 0" rpy="0 0 0"/>
+      <geometry>
+        <mesh filename="package://drone_description/meshes/hokuyo.dae"/>
+      </geometry>
+    </visual>
+    <inertial>
+      <mass value="1e-5" />
+      <origin xyz="0 0 0" rpy="0 0 0"/>
+      <inertia ixx="1e-6" ixy="0" ixz="0" iyy="1e-6" iyz="0" izz="1e-6" />
+    </inertial>
+  </link>
 <link name="base_link">
           <visual>

Commit message: Add files via upload

File: drone_description/urdf/drone.xacro (robot description, xacro)
@@ -3,5 +3,5 @@
 <xacro:include filename="$(find drone_description)/urdf/materials.xacro"/>
 <xacro:include filename="$(find drone_description)/urdf/drone.gazebo"/>
-<link name="foot">
+<link name="base_footprint">
    <visual>
       <origin xyz="0 0 0" rpy="0 0 0" />
@@ -12,11 +12,11 @@
   </link>
   <joint name="base_link_joint" type="fixed">
-    <origin xyz="0.0 0 0.14" rpy="0 0 0" />
-    <parent link="foot"/>
+    <origin xyz="0.0 0 0.15" rpy="0 0 3.14" />
+    <parent link="base_footprint"/>
     <child link="base_link" />
   </joint>
 <joint name="hokuyo_joint" type="fixed">
     <axis xyz="0 1 0" />
-    <origin xyz="0 0 0.2" rpy="0 0 0"/>
+    <origin xyz="0 0 0.14" rpy="0 0 1.57"/>
     <parent link="base_link"/>
     <child link="hokuyo_link"/>
@@ -87,5 +87,5 @@
         <geometry>
          <mesh
-          filename="ppackage://drone_description/meshes/gimbal.stl" />
+          filename="package://drone_description/meshes/gimbal.stl" />
           </geometry>
 </collision>
@@ -104,5 +104,5 @@
 <joint name="camera_joint" type="fixed">
     <axis xyz="1 0 0" />
-    <origin xyz="0 0.175 0.13" rpy="0 0 1.57"/>
+    <origin xyz="0 0.175 0.1" rpy="0 0 1.57"/>
     <parent link="base_link"/>
     <child link="camera_link"/>
